File: kicad-passivator/passivator.sch (KiCad schematic (older format))
At the start: 21 parts, among them P1 In, P2 Out, P3 +9V, P4 -9V, SW1 Cap Selector, SW2.1 SWITCH_INV_SMALL, SW2.2 SWITCH_INV_SMALL, SW2.3 SWITCH_INV_SMALL

Commit message: latest mods, folder cleanup
Signed-off-by: Badscrew <badscrew@dolganoff.com>
Connections:
- net at P1.2 (P2), SW2.1.2: now also SW2.2.1
- net at SW2.1.1: no longer SW2.2.1
Changed lines of the file:
@@
 L GND #PWR01
 U 1 1 554B4199
-P 9450 6300
-F 0 "#PWR01" H 9450 6300 30  0001 C CNN
-F 1 "GND" H 9450 6230 30  0001 C CNN
-F 2 "" H 9450 6300 60  0000 C CNN
-F 3 "" H 9450 6300 60  0000 C CNN
-	1    9450 6300
+P 9450 6200
+F 0 "#PWR01" H 9450 6200 30  0001 C CNN
+F 1 "GND" H 9450 6130 30  0001 C CNN
+F 2 "" H 9450 6200 60  0000 C CNN
+F 3 "" H 9450 6200 60  0000 C CNN
+	1    9450 6200
 	1    0    0    -1
 $EndComp
@@
 $EndComp
 Wire Wire Line
-	8100 6000 8100 6200
-Wire Wire Line
-	8100 6200 9800 6200
-Wire Wire Line
-	9800 6200 9800 6050
-Wire Wire Line
-	9600 6000 9600 6200
-Connection ~ 9600 6200
-Wire Wire Line
-	9300 6050 9300 6200
-Connection ~ 9300 6200
-Wire Wire Line
-	9100 6000 9100 6200
-Connection ~ 9100 6200
-Wire Wire Line
-	8800 6050 8800 6200
-Connection ~ 8800 6200
-Wire Wire Line
-	8600 6000 8600 6200
-Connection ~ 8600 6200
-Wire Wire Line
-	8300 6050 8300 6200
-Connection ~ 8300 6200
+	8100 6000 8100 6100
+Wire Wire Line
+	8100 6100 8300 6100
+Wire Wire Line
+	8300 6100 8600 6100
+Wire Wire Line
+	8600 6100 8800 6100
+Wire Wire Line
+	8800 6100 9100 6100
+Wire Wire Line
+	9100 6100 9300 6100
+Wire Wire Line
+	9300 6100 9450 6100
+Wire Wire Line
+	9450 6100 9600 6100
+Wire Wire Line
+	9600 6100 9800 6100
+Wire Wire Line
+	9800 6100 9800 6050
+Wire Wire Line
+	9600 6000 9600 6100
+Connection ~ 9600 6100
+Wire Wire Line
+	9300 6050 9300 6100
+Connection ~ 9300 6100
+Wire Wire Line
+	9100 6000 9100 6100
+Connection ~ 9100 6100
+Wire Wire Line
+	8800 6050 8800 6100
+Connection ~ 8800 6100
+Wire Wire Line
+	8600 6000 8600 6100
+Connection ~ 8600 6100
+Wire Wire Line
+	8300 6050 8300 6100
+Connection ~ 8300 6100
 Wire Wire Line
 	8100 5600 8100 5500
 Wire Wire Line
-	8000 5500 8300 5500
+	8000 5500 8100 5500
+Wire Wire Line
+	8100 5500 8300 5500
 Wire Wire Line
 	8300 5500 8300 5550
 Wire Wire Line
-	8600 5400 8600 5600
+	8600 5400 8600 5500
+Wire Wire Line
+	8600 5500 8600 5600
 Wire Wire Line
 	8600 5500 8800 5500
@@
 	8800 5500 8800 5550
 Wire Wire Line
-	9100 5300 9100 5600
+	9100 5300 9100 5500
+Wire Wire Line
+	9100 5500 9100 5600
 Wire Wire Line
 	9100 5500 9300 5500
@@
 	9300 5500 9300 5550
 Wire Wire Line
-	9600 5200 9600 5600
+	9600 5200 9600 5500
+Wire Wire Line
+	9600 5500 9600 5600
 Wire Wire Line
 	9600 5500 9800 5500
@@
 Connection ~ 9600 5500
 Wire Wire Line
-	7450 4100 7550 4100
+	7450 4100 7500 4100
+Wire Wire Line
+	7500 4100 7550 4100
 Wire Wire Line
 	8050 4100 8150 4100
 Wire Wire Line
-	9450 6300 9450 6200
-Connection ~ 9450 6200
+	9450 6200 9450 6100
+Connection ~ 9450 6100
 Wire Wire Line
 	10000 4700 10150 4700
@@
 	8450 4750 8450 4850
 Wire Wire Line
-	7300 3800 9550 3800
+	7300 3800 8800 3800
+Wire Wire Line
+	8800 3800 9550 3800
 Wire Wire Line
 	7300 3800 7300 3850
@@
 Connection ~ 7500 4100
 Wire Wire Line
-	9550 3700 9350 3700
-Wire Wire Line
 	9350 4150 9550 4150
 Wire Wire Line
-	6900 3550 10050 3550
+	6900 3550 9350 3550
+Wire Wire Line
+	9350 3550 10050 3550
 Wire Wire Line
 	6900 3550 6900 4900
@@
 	10050 3750 10000 3750
 Wire Wire Line
-	9350 3700 9350 4150
+	9350 3550 9350 4150
 Wire Wire Line
 	10000 4200 10550 4200
@@
 	10150 5550 10350 5550
 Wire Wire Line
-	10350 5750 10150 5750
+	10350 5750 10300 5750
+Wire Wire Line
+	10300 5750 10150 5750
 Wire Wire Line
 	10150 5750 10150 5800
@@
 Wire Wire Line
 	6900 5000 6900 5150
+Connection ~ 9350 3550
 $EndSCHEMATC
